File: core.kicad_sch (KiCad schematic)
At the start: 26 parts, among them U2 W25Q128JVS, U3 RP2040, U4 AZ1117R-3_3TRE1, U6 B5819W_C8598, U7 B5819W_C8598, X1 X322512MSB4SI

Commit message: update
Parts:
- XTRAPI_U2: renamed from U2; LCSC C97521 -> (none)
- renumbered C1 to XTRAPI_C1, C10 to XTRAPI_C10, C11 to XTRAPI_C11, C12 to XTRAPI_C12, C13 to XTRAPI_C13, C14 to XTRAPI_C14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
