File: core.kicad_sch (KiCad schematic)
At the start: 26 parts

Commit message: update
Parts:
- XTRAPI_C1, XTRAPI_C10, XTRAPI_C11, XTRAPI_C12, XTRAPI_C13, XTRAPI_C15, XTRAPI_C16, XTRAPI_C17, XTRAPI_C18, XTRAPI_C2, XTRAPI_C3, XTRAPI_C5, XTRAPI_C6, XTRAPI_C7, XTRAPI_C8, XTRAPI_C9: footprint JLCPCB:C0402 -> XTRAPI_JLC2KiCadLib:C0402
- XTRAPI_C14, XTRAPI_C4: footprint JLCPCB:C1206 -> XTRAPI_JLC2KiCadLib:C1206
- XTRAPI_R2, XTRAPI_R4: footprint JLCPCB:R0402 -> XTRAPI_JLC2KiCadLib:R0402
- XTRAPI_U4: footprint JLCPCB:SOT-89-3_L4.5-W2.5-P1.50-LS4.2-BR -> XTRAPI_JLC2KiCadLib:SOT-89-3_L4.5-W2.5-P1.50-LS4.2-BR
- XTRAPI_U6, XTRAPI_U7: footprint JLCPCB:SOD-123_L2.7-W1.6-LS3.7-RD-1 -> XTRAPI_JLC2KiCadLib:SOD-123_L2.7-W1.6-LS3.7-RD-1
- XTRAPI_X1: footprint JLCPCB:OSC-SMD_4P-L3.2-W2.5-BL -> XTRAPI_JLC2KiCadLib:OSC-SMD_4P-L3.2-W2.5-BL
