File: xtrapico.kicad_sch (KiCad schematic)
At the start: 10 parts, among them U5 X1321FR-2X20-C43D24

Commit message: update
Parts:
- renumbered D1 to XTRA_D1, D2 to XTRA_D2, D3 to XTRA_D3, D4 to XTRA_D4, R1 to XTRA_R1, R3 to XTRA_R3, U5 to XTRA_U5
Changed lines of the file:
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@@
   (symbol (lib_id "JLCPCB_X1321FR-2X20-C43D24:X1321FR-2X20-C43D24") (at 33.02 72.39 0) (unit 1)
     (in_bom yes) (on_board yes) (dnp no)
-    (property "Reference" "U5" (at 33.02 104.14 0)
+    (property "Reference" "XTRA_U5" (at 33.02 104.14 0)
       (effects (font (size 1.27 1.27)))
     )
@@
       (project "xtrapico"
         (path "/84d570ec-9373-46a4-bf76-057b65352f33"
-          (reference "U5") (unit 1)
+          (reference "XTRA_U5") (unit 1)
         )
       )
@@
   (symbol (lib_id "JLCPCB_0402WGF5101TCE:0402WGF5101TCE") (at 97.79 73.66 180) (unit 1)
     (in_bom yes) (on_board yes) (dnp no)
-    (property "Reference" "R3" (at 96.52 76.2 0)
+    (property "Reference" "XTRA_R3" (at 96.52 76.2 0)
       (effects (font (size 1.27 1.27)) (justify right))
     )
@@
       (project "xtrapico"
         (path "/84d570ec-9373-46a4-bf76-057b65352f33"
-          (reference "R3") (unit 1)
+          (reference "XTRA_R3") (unit 1)
         )
       )
@@
   (symbol (lib_id "JLCPCB_0402ESDA-05N:0402ESDA-05N") (at 69.85 130.81 0) (unit 1)
     (in_bom yes) (on_board yes) (dnp no) (fields_autoplaced)
-    (property "Reference" "D4" (at 69.85 124.46 0)
+    (property "Reference" "XTRA_D4" (at 69.85 124.46 0)
       (effects (font (size 1.27 1.27)))
     )
@@
       (project "xtrapico"
         (path "/84d570ec-9373-46a4-bf76-057b65352f33"
-          (reference "D4") (unit 1)
+          (reference "XTRA_D4") (unit 1)
         )
       )
@@
   (symbol (lib_id "JLCPCB_0402ESDA-05N:0402ESDA-05N") (at 69.85 100.33 0) (unit 1)
     (in_bom yes) (on_board yes) (dnp no)
-    (property "Reference" "D1" (at 69.85 93.98 0)
+    (property "Reference" "XTRA_D1" (at 69.85 93.98 0)
       (effects (font (size 1.27 1.27)))
     )
@@
       (project "xtrapico"
         (path "/84d570ec-9373-46a4-bf76-057b65352f33"
-          (reference "D1") (unit 1)
+          (reference "XTRA_D1") (unit 1)
         )
       )
@@
   (symbol (lib_id "JLCPCB_0402WGF5101TCE:0402WGF5101TCE") (at 64.77 66.04 0) (unit 1)
     (in_bom yes) (on_board yes) (dnp no)
-    (property "Reference" "R1" (at 64.77 60.96 0)
+    (property "Reference" "XTRA_R1" (at 64.77 60.96 0)
       (effects (font (size 1.27 1.27)) (justify right))
     )
@@
       (project "xtrapico"
         (path "/84d570ec-9373-46a4-bf76-057b65352f33"
-          (reference "R1") (unit 1)
+          (reference "XTRA_R1") (unit 1)
         )
       )
@@
   (symbol (lib_id "JLCPCB_0402ESDA-05N:0402ESDA-05N") (at 69.85 120.65 0) (unit 1)
     (in_bom yes) (on_board yes) (dnp no) (fields_autoplaced)
-    (property "Reference" "D3" (at 69.85 114.3 0)
+    (property "Reference" "XTRA_D3" (at 69.85 114.3 0)
       (effects (font (size 1.27 1.27)))
     )
@@
       (project "xtrapico"
         (path "/84d570ec-9373-46a4-bf76-057b65352f33"
-          (reference "D3") (unit 1)
+          (reference "XTRA_D3") (unit 1)
         )
       )
@@
   (symbol (lib_id "JLCPCB_0402ESDA-05N:0402ESDA-05N") (at 69.85 110.49 0) (unit 1)
     (in_bom yes) (on_board yes) (dnp no) (fields_autoplaced)
-    (property "Reference" "D2" (at 69.85 104.14 0)
+    (property "Reference" "XTRA_D2" (at 69.85 104.14 0)
       (effects (font (size 1.27 1.27)))
     )
@@
       (project "xtrapico"
         (path "/84d570ec-9373-46a4-bf76-057b65352f33"
-          (reference "D2") (unit 1)
-        )
-      )
+          (reference "XTRA_D2") (unit 1)
+        )
+      )
